Commit message: Update hit box

File: urdf/cameras/rgbd/orbbec_astra_pro_plus.urdf.xacro (robot description, xacro)
@@ -53,7 +53,7 @@
                </visual>
                <collision>
-                    <origin xyz="0.0 0.0 0.0" rpy="0 0 0" />
+                    <origin xyz="-0.0183 0.0 0.0165" rpy="0 0 0" />
                     <geometry>
-                         <box size="0.0730 .2760 0.0720"/>
+                         <box size="0.0370 .1650 0.0350"/>
                     </geometry>
                </collision>
