Commit message: Update for ROS Noetic & Gazebo 11

File: launch/include/sensors_attachments.urdf.xacro (robot description, xacro)
@@ -25,4 +25,7 @@
           <origin xyz="0.26 0 0.05" rpy="0 0 0" />
      </xacro:sensor_realsense_d415>
+     <xacro:sensor_orbbec_astra name="astra" parent="world_link" color="black">
+      <origin xyz="0.23 0 0.15" rpy="0 0 0" />
+     </xacro:sensor_orbbec_astra>
      <!-- IMU -->
      <xacro:sensor_modified_imu name="imu" parent="world_link" color="red"

File: urdf/cameras/rgbd/orbbec_astra.urdf.xacro (robot description, xacro)
@@ -87,5 +87,5 @@
           </link>
           <!-- RGBD sensor for simulation, same as Kinect -->
-          <sensor_orbbec_astra_gazebo/>
+          <xacro:sensor_orbbec_astra_gazebo/>
           <xacro:color_gazebo parent="${name}_link" color="${color}"/>
      </xacro:macro>

Commit message: Fix macro

File: launch/include/sensors_attachments.urdf.xacro (robot description, xacro)
@@ -25,7 +25,7 @@
           <origin xyz="0.26 0 0.05" rpy="0 0 0" />
      </xacro:sensor_realsense_d415>
-     <xacro:sensor_orbbec_astra name="astra" parent="world_link" color="black">
+     <xacro:sensor_orbbec_astra_pro_plus name="astra" parent="world_link" color="black">
       <origin xyz="0.23 0 0.15" rpy="0 0 0" />
-     </xacro:sensor_orbbec_astra>
+     </xacro:sensor_orbbec_astra_pro_plus>
      <!-- IMU -->
      <xacro:sensor_modified_imu name="imu" parent="world_link" color="red"

File: urdf/cameras/camera_sensors.urdf.xacro (robot description, xacro)
@@ -23,4 +23,6 @@
 	<!-- Orbbec Astra -->
 	<xacro:include filename="$(find gazebo_sensor_collection)/urdf/cameras/rgbd/orbbec_astra.urdf.xacro" />
+	<!-- Orbbec Astra Pro Plus -->
+	<xacro:include filename="$(find gazebo_sensor_collection)/urdf/cameras/rgbd/orbbec_astra_pro_plus.urdf.xacro" />
 	<!-- Fotonic E Series -->
 	<xacro:include filename="$(find gazebo_sensor_collection)/urdf/cameras/rgbd/fotonic_e.urdf.xacro" />

File: urdf/cameras/rgbd/orbbec_astra_pro_plus.urdf.xacro (robot description, xacro)
@@ -89,5 +89,5 @@
           </link>
           <!-- RGBD sensor for simulation, same as Kinect -->
-          <xacro:sensor_orbbec_astra_pro_plus_gazebo rgb_w="${rgb_w}" rgb_h="${rgb_h}"/>
+          <xacro:sensor_orbbec_astra_pro_plus_gazebo/>
           <xacro:color_gazebo parent="${name}_link" color="${color}"/>
      </xacro:macro>
@@ -95,5 +95,5 @@
                            Gazebo
      ========================================================= -->
-     <xacro:macro name="sensor_orbbec_astra_pro_plus_gazebo" params="name rgb_w:=640 rgb_h:=480">
+     <xacro:macro name="sensor_orbbec_astra_pro_plus_gazebo">
           <gazebo reference="${name}_link">
                <sensor type="depth" name="${name}">

Commit message: Formatting

File: launch/include/sensors_attachments.urdf.xacro (robot description, xacro)
@@ -1,3 +1,3 @@
-<?xml version="1.0" ?>
+<?xml version="1.0"?>
 <robot name="sensor_suite" xmlns:xacro="http://ros.org/wiki/xacro">
      <!-- ====================================================
@@ -6,5 +6,5 @@
      <xacro:include filename="$(find gazebo_sensor_collection)/urdf/all_sensors.urdf.xacro" />
      <xacro:macro name="world" params="">
-          <link name="world_link"/>
+          <link name="world_link" />
           <gazebo reference="world_link">
                <static>true</static>
@@ -14,7 +14,8 @@
                     Attach and Configure Sensors
      ========================================================= -->
-     <xacro:world/>
+     <xacro:world />
      <!-- LiDAR sensor_hokuyo_ust10lx -->
-     <!-- <xacro:sensor_hokuyo_ust10lx name="hokuyo" parent="world_link" color="black" visualize="true">
+     <!-- <xacro:sensor_hokuyo_ust10lx name="hokuyo" parent="world_link" color="black"
+     visualize="true">
           <origin xyz="0.22 0 0.173" rpy="0 0 0"/>
      </xacro:sensor_hokuyo_ust10lx> -->
@@ -26,34 +27,34 @@
      </xacro:sensor_realsense_d415>
      <xacro:sensor_orbbec_astra_pro_plus name="astra" parent="world_link" color="black">
-      <origin xyz="0.23 0 0.15" rpy="0 0 0" />
+          <origin xyz="0.23 0 0.15" rpy="0 0 0" />
      </xacro:sensor_orbbec_astra_pro_plus>
      <!-- IMU -->
      <xacro:sensor_modified_imu name="imu" parent="world_link" color="red"
-                    update_rate="50.0"
-                    noise="0.005"
-                    yaw_offset="0.0"
-                    yaw_drift="0.02"
-                    yaw_noise="0.01"
-                    rate_offset="0.0 0.0 0.0"
-                    rate_drift="0.002 0.002 0.002"
-                    rate_noise="0.001 0.001 0.001"
-                    accel_offset="0.0 0.0 0.0"
-                    accel_drift="0.005 0.005 0.005"
-                    accel_noise="0.005 0.005 0.005">
-          <origin xyz="0 0 0" rpy="0 0 0"/>
+          update_rate="50.0"
+          noise="0.005"
+          yaw_offset="0.0"
+          yaw_drift="0.02"
+          yaw_noise="0.01"
+          rate_offset="0.0 0.0 0.0"
+          rate_drift="0.002 0.002 0.002"
+          rate_noise="0.001 0.001 0.001"
+          accel_offset="0.0 0.0 0.0"
+          accel_drift="0.005 0.005 0.005"
+          accel_noise="0.005 0.005 0.005">
+          <origin xyz="0 0 0" rpy="0 0 0" />
      </xacro:sensor_modified_imu>
      <!-- GPS w/ Variable Dropouts-->
      <xacro:sensor_gps_with_dropout name="gps" parent="world_link" color="white"
-                    ref_lat="40.1021496545"
-                    ref_long="-88.2267974168"
-                    ref_head="90.0"
-                    update_rate="10.0"
-                    drift="0.0"
-                    noise="0.001"
-                    vel_drift="0.00001"
-                    vel_noise="0.00001">
-          <origin xyz="-0.14 0 0.12" rpy="0 0 0"/>
+          ref_lat="40.1021496545"
+          ref_long="-88.2267974168"
+          ref_head="90.0"
+          update_rate="10.0"
+          drift="0.0"
+          noise="0.001"
+          vel_drift="0.00001"
+          vel_noise="0.00001">
+          <origin xyz="-0.14 0 0.12" rpy="0 0 0" />
      </xacro:sensor_gps_with_dropout>
      <!-- Simple Simulated Battery -->
-     <xacro:sensor_battery_approx/>
+     <xacro:sensor_battery_approx />
 </robot>

File: urdf/cameras/rgbd/orbbec_astra_pro_plus.urdf.xacro (robot description, xacro)
@@ -1,11 +1,11 @@
 <?xml version="1.0"?>
 <robot name="sensor_orbbec_astra_pro_plus" xmlns:xacro="http://ros.org/wiki/xacro">
-     <xacro:include filename="$(find gazebo_sensor_collection)/urdf/includes/materials.urdf.xacro"/>
-     <xacro:property name="orbbec_astra_pro_plus_scale" value="1.0"/>
+     <xacro:include filename="$(find gazebo_sensor_collection)/urdf/includes/materials.urdf.xacro" />
+     <xacro:property name="orbbec_astra_pro_plus_scale" value="1.0" />
      <!-- RGB sensor - cam -->
      <!-- THESE MIGHT NEED TO CHANGE IF THE RESOLUTION IS NOT 640x480 -->
-     <xacro:property name="orbbec_astra_pro_plus_rel_rgb_px"   value="0.0" />
-     <xacro:property name="orbbec_astra_pro_plus_rel_rgb_py"   value="-0.0125" />
-     <xacro:property name="orbbec_astra_pro_plus_rel_rgb_pz"   value="-0.0150" />
+     <xacro:property name="orbbec_astra_pro_plus_rel_rgb_px" value="0.0" />
+     <xacro:property name="orbbec_astra_pro_plus_rel_rgb_py" value="-0.0125" />
+     <xacro:property name="orbbec_astra_pro_plus_rel_rgb_pz" value="-0.0150" />
      <!-- IR sensor - depth -->
      <xacro:property name="orbbec_astra_pro_plus_depth_rel_rgb_px" value="0.0" />
@@ -14,8 +14,9 @@
      <xacro:property name="M_PI" value="3.1415926535897931" />
      <!--  -->
-     <xacro:macro name="sensor_orbbec_astra_pro_plus" params="name parent *origin color rgb_w:=640 rgb_h:=480">
+     <xacro:macro name="sensor_orbbec_astra_pro_plus"
+          params="name parent *origin color rgb_w:=640 rgb_h:=480">
           <joint name="${name}_rgb_joint" type="fixed">
                <xacro:insert_block name="origin" />
-               <parent link="${parent}"/>
+               <parent link="${parent}" />
                <child link="${name}_rgb_frame" />
           </joint>
@@ -40,20 +41,24 @@
           </link>
           <joint name="${name}_joint" type="fixed">
-               <origin xyz="${orbbec_astra_pro_plus_rel_rgb_px} ${orbbec_astra_pro_plus_rel_rgb_py} ${orbbec_astra_pro_plus_rel_rgb_pz}" rpy="0.0 0 0"/>
-               <parent link="${name}_rgb_frame"/>
-               <child link="${name}_link"/>
+               <origin
+                    xyz="${orbbec_astra_pro_plus_rel_rgb_px} ${orbbec_astra_pro_plus_rel_rgb_py} ${orbbec_astra_pro_plus_rel_rgb_pz}"
+                    rpy="0.0 0 0" />
+               <parent link="${name}_rgb_frame" />
+               <child link="${name}_link" />
           </joint>
           <link name="${name}_link">
                <visual>
-                    <origin xyz="0 0 0" rpy="0 0 0"/>
+                    <origin xyz="0 0 0" rpy="0 0 0" />
                     <geometry>
-                         <mesh filename="package://gazebo_sensor_collection/meshes/cameras/orbbec/orbbec_astra.dae" scale="${orbbec_astra_pro_plus_scale} ${orbbec_astra_pro_plus_scale} ${orbbec_astra_pro_plus_scale}"/>
+                         <mesh
+                              filename="package://gazebo_sensor_collection/meshes/cameras/orbbec/orbbec_astra.dae"
+                              scale="${orbbec_astra_pro_plus_scale} ${orbbec_astra_pro_plus_scale} ${orbbec_astra_pro_plus_scale}" />
                     </geometry>
-                    <xacro:color_material color="${color}"/>
+                    <xacro:color_material color="${color}" />
                </visual>
                <collision>
                     <origin xyz="-0.0183 0.0 0.0165" rpy="0 0 0" />
                     <geometry>
-                         <box size="0.0370 .1650 0.0350"/>
+                         <box size="0.0370 .1650 0.0350" />
                     </geometry>
                </collision>
@@ -61,9 +66,12 @@
                     <mass value="0.564" />
                     <origin xyz="0 0 0" />
-                    <inertia ixx="0.003881243" ixy="0.0" ixz="0.0" iyy="0.000498940" iyz="0.0" izz="0.003879257" />
+                    <inertia ixx="0.003881243" ixy="0.0" ixz="0.0" iyy="0.000498940" iyz="0.0"
+                         izz="0.003879257" />
                </inertial>
           </link>
           <joint name="${name}_depth_joint" type="fixed">
-               <origin xyz="${orbbec_astra_pro_plus_depth_rel_rgb_px} ${orbbec_astra_pro_plus_depth_rel_rgb_py} ${orbbec_astra_pro_plus_depth_rel_rgb_pz}" rpy="0 0 0" />
+               <origin
+                    xyz="${orbbec_astra_pro_plus_depth_rel_rgb_px} ${orbbec_astra_pro_plus_depth_rel_rgb_py} ${orbbec_astra_pro_plus_depth_rel_rgb_pz}"
+                    rpy="0 0 0" />
                <parent link="${name}_rgb_frame" />
                <child link="${name}_depth_frame" />
@@ -89,6 +97,6 @@
           </link>
           <!-- RGBD sensor for simulation, same as Kinect -->
-          <xacro:sensor_orbbec_astra_pro_plus_gazebo/>
-          <xacro:color_gazebo parent="${name}_link" color="${color}"/>
+          <xacro:sensor_orbbec_astra_pro_plus_gazebo />
+          <xacro:color_gazebo parent="${name}_link" color="${color}" />
      </xacro:macro>
      <!-- ====================================================
@@ -129,5 +137,6 @@
                          <distortion_t2>0.0</distortion_t2>
                          <pointCloudCutoff>0.4</pointCloudCutoff> <!-- Shouldn't this be 0.6-->
-                         <!-- https://github.com/osrf/gazebo_tutorials/blob/master/ros_depth_camera/tutorial.md  -->
+                         <!--
+                         https://github.com/osrf/gazebo_tutorials/blob/master/ros_depth_camera/tutorial.md  -->
                          <!-- https://shop.orbbec3d.com/Astra-Pro-Plus -->
                     </plugin>
